File: rev.04/IR-endstop-04.sch (KiCad schematic (older format))
At the start: 6 parts, among them P1 CONN_01X03, Q1 2N7002KT1G, U1 EE-SX1103

Commit message: pcb rev0.4
Parts:
- added D2: BAT54KFILM, ok1hra:SOD-523-ShortSilk, symbol IR-endstop-04-rescue:D_ALT-device-DLP-control-rescue-DLP-control-04-rescue-DLP-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
- added R4: 56k, Resistors_SMD:R_0402, symbol device:R
- Q1: req (none) -> 60V/0,38A/2.5Ω/ESD Protected
- R2, R3: footprint Resistors_SMD:R_0603 -> Resistors_SMD:R_0402
Connections:
- net labels added: GND
- wire segments 24 -> 29
Other:
- note added: "0,32V"
- note added: "11mA"
- note added: "Changelog\n--------\nrev 0.4\n- add R4\nrev 0.3\n- add D2"
Changed lines of the file:
@@
 EESchema Schematic File Version 4
-LIBS:IR-endstop-01-cache
-EELAYER 26 0
+EELAYER 30 0
 EELAYER END
 $Descr A4 11693 8268
@@
 Sheet 1 1
 Title "IR sensor"
-Date "2019-02-12"
-Rev "0.1"
-Comp "PRUSA RESEARCH s.r.o"
-Comment1 "#ok1hra"
-Comment2 ""
-Comment3 ""
+Date "2019-07-04"
+Rev "0.4"
+Comp "Prusa Development a.s."
+Comment1 "http://creativecommons.org/licenses/by-sa/4.0/"
+Comment2 "Licensed under the Attribution-ShareAlike 4.0 International (CC BY-SA 4.0)"
+Comment3 "#ok1hra"
 Comment4 ""
 $EndDescr
@@
 L conn:CONN_01X03 P1
 U 1 1 5BD70990
-P 7050 3575
-F 0 "P1" H 7128 3616 50  0000 L CNN
-F 1 "CONN_01X03" H 7128 3525 50  0000 L CNN
-F 2 "Pin_Headers:Pin_Header_Angled_1x03" H 7050 3575 50  0001 C CNN
-F 3 "" H 7050 3575 50  0001 C CNN
-F 4 "" H 7050 3575 50  0001 C CNN "alternative"
-	1    7050 3575
+P 7525 3575
+F 0 "P1" H 7603 3616 50  0000 L CNN
+F 1 "CONN_01X03" H 7603 3525 50  0000 L CNN
+F 2 "Pin_Headers:Pin_Header_Angled_1x03" H 7525 3575 50  0001 C CNN
+F 3 "" H 7525 3575 50  0001 C CNN
+F 4 "" H 7525 3575 50  0001 C CNN "alternative"
+	1    7525 3575
 	1    0    0    -1
 $EndComp
@@
 Wire Wire Line
 	4300 3875 4350 3875
-Text Notes 6700 3675 0    61   ~ 0
+Text Notes 7175 3675 0    61   ~ 0
 +5V\nOUT\nGND
 $Comp
@@
 F 0 "R2" V 5250 3675 50  0000 C CNN
 F 1 "10k" V 5400 3675 50  0000 C CNN
-F 2 "Resistors_SMD:R_0603" V 5330 3675 50  0001 C CNN
+F 2 "Resistors_SMD:R_0402" V 5330 3675 50  0001 C CNN
 F 3 "" H 5400 3675 50  0001 C CNN
 F 4 "0,1W/1%" V 5300 3675 28  0000 C CNN "req"
@@
 Connection ~ 5400 4325
 Wire Wire Line
-	6025 4325 6575 4325
+	6025 4325 7050 4325
 Wire Wire Line
-	6575 4325 6575 3675
+	7050 4325 7050 4175
 Wire Wire Line
-	6575 3675 6850 3675
+	7050 3675 7325 3675
 Connection ~ 6025 4325
 Wire Wire Line
-	6850 3575 6025 3575
+	7325 3575 6550 3575
 Wire Wire Line
 	6025 3575 6025 3625
@@
 F 0 "R3" V 5600 3575 50  0000 C CNN
 F 1 "10k" V 5750 3575 50  0000 C CNN
-F 2 "Resistors_SMD:R_0603" V 5680 3575 50  0001 C CNN
+F 2 "Resistors_SMD:R_0402" V 5680 3575 50  0001 C CNN
 F 3 "" H 5750 3575 50  0001 C CNN
 F 4 "0,1W/1%" V 5650 3575 28  0000 C CNN "req"
@@
 Wire Wire Line
 	5500 3475 5400 3475
+Text Notes 4275 3875 1    50   ~ 0
+11mA
+Text Notes 5275 3975 0    50   ~ 0
+0,32V
 $Comp
 L transistors:2N7002 Q1
@@
 F 2 "TO_SOT_Packages_SMD:SOT-23" H 6125 3750 50  0001 L CIN
 F 3 "" H 6116 3734 50  0001 L CNN
+F 4 "60V/0,38A/2.5Ω/ESD Protected" H 6475 3700 28  0000 C CNN "req"
 	1    5925 3825
 	1    0    0    -1
@@
 	5400 4325 6025 4325
 Wire Wire Line
-	6850 3475 5500 3475
+	7325 3475 5500 3475
 Connection ~ 5500 3475
+Wire Wire Line
+	7050 3875 7050 3675
+$Comp
+L IR-endstop-04-rescue:D_ALT-device-DLP-control-rescue-DLP-control-04-rescue-DLP-control-05-rescue-SL1-control-05b-rescue-SL-controller-06-rescue-SL-controller-06b-rescue-SL-controller-06c-rescue-IR-endstop-03-rescue-IR-endstop-03b-rescue D2
+U 1 1 5D0C3FD7
+P 7050 4025
+F 0 "D2" V 6975 4125 50  0000 L CNN
+F 1 "BAT54KFILM" V 7050 4125 50  0000 L CNN
+F 2 "ok1hra:SOD-523-ShortSilk" H 7050 4025 50  0001 C CNN
+F 3 "" H 7050 4025 50  0001 C CNN
+F 4 "400mV@10mA/40V/0,3A" V 7125 4125 28  0000 L CNN "req"
+	1    7050 4025
+	0    1    1    0
+$EndComp
+Text Label 6200 4325 0    50   ~ 0
+GND
+Text Notes 6100 7450 0    50   ~ 0
+Changelog\n--------\nrev 0.4\n- add R4\nrev 0.3\n- add D2
+$Comp
+L device:R R4
+U 1 1 5D1DA941
+P 6800 3675
+F 0 "R4" V 6650 3675 50  0000 C CNN
+F 1 "56k" V 6800 3675 50  0000 C CNN
+F 2 "Resistors_SMD:R_0402" V 6730 3675 50  0001 C CNN
+F 3 "" H 6800 3675 50  0001 C CNN
+F 4 "0,1W/1%" V 6700 3675 28  0000 C CNN "req"
+	1    6800 3675
+	0    1    -1   0
+$EndComp
+Wire Wire Line
+	6650 3675 6550 3675
+Wire Wire Line
+	6550 3675 6550 3575
+Connection ~ 6550 3575
+Wire Wire Line
+	6550 3575 6025 3575
+Wire Wire Line
+	6950 3675 7050 3675
+Connection ~ 7050 3675
 $EndSCHEMATC
